Commit message: Updated main and removed excess files

File: robot-endpoint/yahboom_files/urdf/dofbot.urdf (robot description, URDF)
Before this commit: robot arm, 6 links, 5 joints
Links:
- link base_link: geometry collision mesh filename=package://arm_moveit/meshes/base_link.STL; visual mesh filename=package://arm_moveit/meshes/base_link.STL
- link link1: geometry collision mesh filename=package://arm_moveit/meshes/link1.STL; visual mesh filename=package://arm_moveit/meshes/link1.STL
- link link2: geometry collision mesh filename=package://arm_moveit/meshes/link2.STL; visual mesh filename=package://arm_moveit/meshes/link2.STL
- link link3: geometry collision mesh filename=package://arm_moveit/meshes/link3.STL; visual mesh filename=package://arm_moveit/meshes/link3.STL
- link link4: geometry collision mesh filename=package://arm_moveit/meshes/link4.STL; visual mesh filename=package://arm_moveit/meshes/link4.STL
- link link5: geometry collision mesh filename=package://arm_moveit/meshes/link5.STL; visual mesh filename=package://arm_moveit/meshes/link5.STL
